File: hardware/LineLight-1.kicad_sch (KiCad schematic)
At the start: 23 parts, among them J1 AUDIO_IN_TRS, J2 AUDIO_THRU, J3 ProMicro_Left, J4 ProMicro_Right, J5 Lamp_OUT, J6 Power_12V, Q1 AO3400A, U1 LM358

Commit message: Retarget firmware stack to FTDI-flashed Pro Mini
Other:
- note added: "ADC → Pro Mini 5V"
- note added: "Finish by wiring pins to labels on a 2.54 mm grid. Annotate, then Assign Footprints. Pro Mini pins: map A0, D9, +5V, GND accordingly."
- note removed: "ADC → Pro Micro 5V"
- note removed: "Finish by wiring pins to labels on a 2.54 mm grid. Annotate, then Assign Footprints. Pro Micro pins: map A0, D9, +5V, GND accordingly."
Changed lines of the file:
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@@
 (text "Audio I/O (TRS/through)" (at 20.00 20.00 0) (effects (font (size 2.2 2.2))))
 (text "Op-Amp envelope detector + bias" (at 20.00 60.00 0) (effects (font (size 2.2 2.2))))
-(text "ADC → Pro Micro 5V" (at 120.00 60.00 0) (effects (font (size 2.2 2.2))))
+(text "ADC → Pro Mini 5V" (at 120.00 60.00 0) (effects (font (size 2.2 2.2))))
 (text "Lamp driver (logic-level N-MOSFET)" (at 120.00 20.00 0) (effects (font (size 2.2 2.2))))
 (text "User controls (pots set FFT window)" (at 20.00 100.00 0) (effects (font (size 2.2 2.2))))
@@
 (text "Finish by wiring pins to labels on a 2.54 mm grid.
 Annotate, then Assign Footprints.
-Pro Micro pins: map A0, D9, +5V, GND accordingly." (at 110.00 96.00 0) (effects (font (size 1.4 1.4))))
+Pro Mini pins: map A0, D9, +5V, GND accordingly." (at 110.00 96.00 0) (effects (font (size 1.4 1.4))))
   (path
     "/"
